Commit message: work

File: basic_mobile_robot/models/basic_mobile_bot_v2.urdf (robot description, URDF)
Before this commit: robot basic_mobile_bot, 6 links, 5 joints
Links:
- link base_link: geometry collision box size=${base_length} ${base_width} ${base_height}; visual mesh filename=package://basic_mobile_robot/meshes/robot_base.stl
