Commit message: added the SDP 12 URDF

File: basic_mobile_robot/models/robo_holly.urdf (robot description, URDF)
Before this commit: robot basic_mobile_bot, 6 links, 5 joints
Links:
- removed link front_caster
- link base_link: geometry collision box size=${base_length} ${base_width} ${base_height}; visual mesh filename=package://basic_mobile_robot/meshes/robot_base.stl
Joints:
- removed joint caster_joint

Commit message: to do SDF file 11/14/23

File: basic_mobile_robot/models/robo_holly.urdf (robot description, URDF)
Before this commit: robot basic_mobile_bot, 5 links, 4 joints
Links:
- link base_link: geometry collision box size=${base_length} ${base_width} ${base_height}; visual box size=${base_length} ${base_width} ${base_height}
- link lidar_link: geometry collision cylinder length=0.057 radius=0.0762; visual cylinder length=0.057 radius=0.0762
Joints:
- joint gps_joint: origin xyz=0.10 0 0.05 rpy=0 0 0 -> xyz=0.10 0 0.0 rpy=0 0 0
- joint imu_joint: origin xyz=-0.10 0 0.05 rpy=0 0 0 -> xyz=-0.10 0 0.0 rpy=0 0 0
- joint lidar_joint: origin xyz=0.215 0 0.13 rpy=0 0 0 -> xyz=0 0 0.05 rpy=0 0 0

Commit message: work in progress

File: basic_mobile_robot/models/robo_holly.urdf (robot description, URDF)
Before this commit: robot basic_mobile_bot, 5 links, 4 joints
Links:
- link lidar_link: geometry collision cylinder length=0.057 radius=0.0381; visual cylinder length=0.057 radius=0.0381
Joints:
- joint lidar_joint: origin xyz=0 0 0.05 rpy=0 0 0 -> xyz=0 0 -0.01 rpy=0 0 1.57

Commit message: navigation working!! Checkpoint 1

File: basic_mobile_robot/models/robo_holly.urdf (robot description, URDF)
Before this commit: robot robo_holly, 5 links, 4 joints
Joints:
- joint lidar_joint: origin xyz=0 0 -0.01 rpy=0 0 1.57 -> xyz=-0.1905 0 0.381 rpy=0 0 0

Commit message: navigation all set up! Fine tuning todo

File: basic_mobile_robot/models/robo_holly.urdf (robot description, URDF)
Before this commit: robot robo_holly, 5 links, 4 joints
Joints:
- joint lidar_joint: origin xyz=-0.1905 0 0.381 rpy=0 0 0 -> xyz=-0.1905 0 0.381 rpy=0 0 1.57

Commit message: better slam

File: basic_mobile_robot/models/robo_holly.urdf (robot description, URDF)
Before this commit: robot robo_holly, 5 links, 4 joints
Joints:
- joint lidar_joint: origin xyz=-0.1905 0 0.381 rpy=0 0 1.57 -> xyz=-0.1905 0 0.381 rpy=0 0 0

Commit message: work in progress 11/29

File: basic_mobile_robot/models/robo_holly.urdf (robot description, URDF)
Before this commit: robot robo_holly, 5 links, 4 joints
Links:
- removed link gps_link
Joints:
- removed joint gps_joint
- joint imu_joint: origin xyz=-0.10 0 0.0 rpy=0 0 0 -> xyz=-0.0254 0 0.1524 rpy=3.14159 0 3.14159
- joint lidar_joint: origin xyz=-0.1905 0 0.381 rpy=0 0 0 -> xyz=0.1905 0 0.381 rpy=0 0 3.14159

File: install/basic_mobile_robot/share/basic_mobile_robot/models/robo_holly.urdf (robot description, URDF)
Before this commit: robot robo_holly, 5 links, 4 joints
Links:
- removed link gps_link
Joints:
- removed joint gps_joint
- joint imu_joint: origin xyz=-0.10 0 0.0 rpy=0 0 0 -> xyz=-0.0254 0 0.1524 rpy=3.14159 0 3.14159
- joint lidar_joint: origin xyz=-0.1905 0 0.381 rpy=0 0 0 -> xyz=0.1905 0 0.381 rpy=0 0 3.14159

Commit message: fixed map jump errors. Need to figure out turning

File: basic_mobile_robot/models/robo_holly.urdf (robot description, URDF)
Before this commit: robot robo_holly, 3 links, 2 joints
Joints:
- joint lidar_joint: origin xyz=0.1905 0 0.381 rpy=0 0 3.14159 -> xyz=0.1905 0 0.381 rpy=0 0 0

Commit message: checkpoint 1 2/12/24

File: basic_mobile_robot/models/robo_holly.urdf (robot description, URDF)
Before this commit: robot robo_holly, 3 links, 2 joints
Joints:
- joint lidar_joint: origin xyz=0.1905 0 0.381 rpy=0 0 0 -> xyz=-0.03 0 0.235 rpy=0 0 0

Commit message: checkpoint updated URDF and functionality

File: basic_mobile_robot/models/robo_holly.urdf (robot description, URDF)
Before this commit: robot robo_holly, 3 links, 2 joints
Joints:
- joint imu_joint: origin xyz=-0.0254 0 0.1524 rpy=3.14159 0 3.14159 -> xyz=-0.044 0 0.21 rpy=3.14159 0 3.14159
- joint lidar_joint: origin xyz=-0.03 0 0.235 rpy=0 0 0 -> xyz=-0.0254 0 0.254 rpy=0 0 0

Commit message: update URDF checkpoint 2

File: basic_mobile_robot/models/robo_holly.urdf (robot description, URDF)
Before this commit: robot robo_holly, 3 links, 2 joints
Joints:
- joint imu_joint: origin xyz=-0.044 0 0.21 rpy=3.14159 0 3.14159 -> xyz=-0.0254 0 0.03 rpy=3.14159 0 3.14159
