Commit message: added physical robot ros2 control packages

File: control_ws/install/my_bot/share/my_bot/description/ros2_control.xacro (robot description, xacro)
@@ -1,24 +1,18 @@
 <?xml version="1.0"?>
 <robot xmlns:xacro="http://www.ros.org/wiki/xacro" name="robot">
-    <ros2_control name="GazeboSystem" type="system">
+    <ros2_control name="RealRobot" type="system">
+        <!-- <hardware>
+            <plugin>diffdrive_arduino/DiffDriveArduino</plugin>
+            <param name="left_wheel_name">drivewhl_lf_joint</param>
+            <param name="right_wheel_name">drivewhl_rf_joint</param>
+            <param name="loop_rate">30</param>
+            <param name="device">/dev/ttyACM1</param>
+            <param name="baud_rate">115200</param>
+            <param name="timeout">0.01</param>
+            <param name="enc_counts_per_rev">3436</param>
+        </hardware> -->
         <hardware>
             <plugin>gazebo_ros2_control/GazeboSystem</plugin>
         </hardware>
-        <!-- <joint name="left_wheel_joint">
-            <command_interface name="velocity">
-                <param name="min">-10</param>
-                <param name="max">10</param>
-            </command_interface>
-            <state_interface name="position" />
-            <state_interface name="velocity" />
-        </joint>
-        <joint name="right_wheel_joint">
-            <command_interface name="velocity">
-                <param name="min">-10</param>
-                <param name="max">10</param>
-            </command_interface>
-            <state_interface name="velocity" />
-            <state_interface name="position" />
-        </joint> -->
         <joint name="drivewhl_lf_joint">
             <command_interface name="velocity">
