Commit message: update to new chassis. Checkpoint 1

File: navphy_ws/basic_mobile_robot/models/robo_holly.urdf (robot description, URDF)
Before this commit: robot robo_holly, 3 links, 2 joints
Joints:
- joint imu_joint: origin xyz=-0.0254 0 0.03 rpy=3.14159 0 3.14159 -> xyz=-0.0254 0 0.03 rpy=3.14159 0 0

Commit message: update to new robot 3/4/23

File: navphy_ws/basic_mobile_robot/models/robo_holly.urdf (robot description, URDF)
Before this commit: robot robo_holly, 3 links, 2 joints
Joints:
- joint imu_joint: origin xyz=-0.0254 0 0.03 rpy=3.14159 0 0 -> xyz=-0.0254 0 0.03 rpy=0 0 3.14159

Commit message: FPR testing changes 4/24/24

File: navphy_ws/basic_mobile_robot/models/robo_holly.urdf (robot description, URDF)
Before this commit: robot robo_holly, 3 links, 2 joints
Joints:
- joint imu_joint: origin xyz=-0.0254 0 0.03 rpy=0 0 3.14159 -> xyz=-0.03 0 0.03 rpy=0 0 -1.5707963267949

Commit message: checkpoint working pre demo day

File: navphy_ws/basic_mobile_robot/models/robo_holly.urdf (robot description, URDF)
Before this commit: robot robo_holly, 3 links, 2 joints
Joints:
- joint lidar_joint: origin xyz=-0.0254 0 0.254 rpy=0 0 0 -> xyz=-0.0254 0 0.254 rpy=0 0 3.14
